File: RPHAT_nucleo.kicad_pcb (KiCad board)
At the start: 2 copper layers, 2 parts, among them J1 Raspberry_Pi_2_3, U1 NUCLEO-F446RE

Commit message: to 6.0
Other:
- net class Default removed

Commit message: on
Parts:
- added U2: MCP2551-I-SN, Package_SO:SOIC-8_3.9x4.9mm_P1.27mm, F.Cu at (154.3, 96.5)
Connections:
- net Net-(U1-Pad54) renamed /nuCAN2_TX
- net Net-(U1-Pad68) renamed /nuCAN2_RX
- J1 pad 1: Net-(J1-Pad1) -> +3V3
- J1 pad 10: Net-(J1-Pad10) -> /Serial_nu_to_rp
- J1 pad 11: Net-(J1-Pad11) -> unconnected-(J1-Pad11)
- J1 pad 12: Net-(J1-Pad12) -> unconnected-(J1-Pad12)
- J1 pad 13: Net-(J1-Pad13) -> unconnected-(J1-Pad13)
- J1 pad 14: Net-(J1-Pad14) -> unconnected-(J1-Pad14)
- J1 pad 15: Net-(J1-Pad15) -> unconnected-(J1-Pad15)
- J1 pad 16: Net-(J1-Pad16) -> unconnected-(J1-Pad16)
- J1 pad 17: Net-(J1-Pad17) -> +3V3
- J1 pad 18: Net-(J1-Pad18) -> unconnected-(J1-Pad18)
- J1 pad 19: Net-(J1-Pad19) -> unconnected-(J1-Pad19)
- J1 pad 2: Net-(J1-Pad2) -> +5V
- J1 pad 20: Net-(J1-Pad20) -> unconnected-(J1-Pad20)
- J1 pad 21: Net-(J1-Pad21) -> unconnected-(J1-Pad21)
- J1 pad 22: Net-(J1-Pad22) -> unconnected-(J1-Pad22)
- J1 pad 23: Net-(J1-Pad23) -> unconnected-(J1-Pad23)
- J1 pad 24: Net-(J1-Pad24) -> unconnected-(J1-Pad24)
- J1 pad 25: Net-(J1-Pad25) -> unconnected-(J1-Pad25)
- J1 pad 26: Net-(J1-Pad26) -> unconnected-(J1-Pad26)
- J1 pad 27: Net-(J1-Pad27) -> unconnected-(J1-Pad27)
- J1 pad 28: Net-(J1-Pad28) -> unconnected-(J1-Pad28)
- J1 pad 29: Net-(J1-Pad29) -> unconnected-(J1-Pad29)
- J1 pad 3: Net-(J1-Pad3) -> unconnected-(J1-Pad3)
- J1 pad 30: Net-(J1-Pad30) -> unconnected-(J1-Pad30)
- J1 pad 31: Net-(J1-Pad31) -> unconnected-(J1-Pad31)
- J1 pad 32: Net-(J1-Pad32) -> unconnected-(J1-Pad32)
- J1 pad 33: Net-(J1-Pad33) -> unconnected-(J1-Pad33)
- J1 pad 34: Net-(J1-Pad34) -> unconnected-(J1-Pad34)
- J1 pad 35: Net-(J1-Pad35) -> unconnected-(J1-Pad35)
- J1 pad 36: Net-(J1-Pad36) -> unconnected-(J1-Pad36)
- J1 pad 37: Net-(J1-Pad37) -> unconnected-(J1-Pad37)
- J1 pad 38: Net-(J1-Pad38) -> unconnected-(J1-Pad38)
- J1 pad 39: Net-(J1-Pad39) -> unconnected-(J1-Pad39)
- J1 pad 4: Net-(J1-Pad4) -> +5V
- J1 pad 40: Net-(J1-Pad40) -> unconnected-(J1-Pad40)
- J1 pad 5: Net-(J1-Pad5) -> unconnected-(J1-Pad5)
- J1 pad 6: Net-(J1-Pad6) -> unconnected-(J1-Pad6)
- J1 pad 7: Net-(J1-Pad7) -> unconnected-(J1-Pad7)
- J1 pad 8: Net-(J1-Pad8) -> /Serial_rp_to_nu
- J1 pad 9: Net-(J1-Pad9) -> unconnected-(J1-Pad9)
- U1 pad 1: Net-(U1-Pad1) -> unconnected-(U1-Pad1)
- U1 pad 10: Net-(U1-Pad10) -> unconnected-(U1-Pad10)
- U1 pad 11: Net-(U1-Pad11) -> unconnected-(U1-Pad11)
- U1 pad 12: Net-(U1-Pad12) -> unconnected-(U1-Pad12)
- U1 pad 13: Net-(U1-Pad13) -> unconnected-(U1-Pad13)
- U1 pad 14: Net-(U1-Pad14) -> unconnected-(U1-Pad14)
- U1 pad 15: Net-(U1-Pad15) -> unconnected-(U1-Pad15)
- U1 pad 16: Net-(U1-Pad16) -> unconnected-(U1-Pad16)
- U1 pad 17: Net-(U1-Pad17) -> unconnected-(U1-Pad17)
- U1 pad 18: Net-(U1-Pad18) -> unconnected-(U1-Pad18)
- U1 pad 19: Net-(U1-Pad19) -> unconnected-(U1-Pad19)
- U1 pad 2: Net-(U1-Pad2) -> unconnected-(U1-Pad2)
- U1 pad 20: Net-(U1-Pad20) -> unconnected-(U1-Pad20)
- U1 pad 21: Net-(U1-Pad21) -> unconnected-(U1-Pad21)
- U1 pad 22: Net-(U1-Pad22) -> unconnected-(U1-Pad22)
- U1 pad 23: Net-(U1-Pad23) -> unconnected-(U1-Pad23)
- U1 pad 24: Net-(U1-Pad24) -> unconnected-(U1-Pad24)
- U1 pad 25: Net-(U1-Pad25) -> unconnected-(U1-Pad25)
- U1 pad 26: Net-(U1-Pad26) -> unconnected-(U1-Pad26)
- U1 pad 27: Net-(U1-Pad27) -> unconnected-(U1-Pad27)
- U1 pad 28: Net-(U1-Pad28) -> unconnected-(U1-Pad28)
- U1 pad 29: Net-(U1-Pad29) -> unconnected-(U1-Pad29)
- U1 pad 3: Net-(U1-Pad3) -> unconnected-(U1-Pad3)
- U1 pad 30: Net-(U1-Pad30) -> unconnected-(U1-Pad30)
- U1 pad 31: Net-(U1-Pad31) -> unconnected-(U1-Pad31)
- U1 pad 32: Net-(U1-Pad32) -> unconnected-(U1-Pad32)
- U1 pad 33: Net-(U1-Pad33) -> unconnected-(U1-Pad33)
- U1 pad 34: Net-(U1-Pad34) -> unconnected-(U1-Pad34)
- U1 pad 35: Net-(U1-Pad35) -> unconnected-(U1-Pad35)
- U1 pad 36: Net-(U1-Pad36) -> unconnected-(U1-Pad36)
- U1 pad 37: Net-(U1-Pad37) -> unconnected-(U1-Pad37)
- U1 pad 38: Net-(U1-Pad38) -> unconnected-(U1-Pad38)
- U1 pad 39: Net-(U1-Pad39) -> unconnected-(U1-Pad39)
- U1 pad 4: Net-(U1-Pad4) -> unconnected-(U1-Pad4)
- U1 pad 40: Net-(U1-Pad40) -> unconnected-(U1-Pad40)
- U1 pad 41: Net-(U1-Pad41) -> unconnected-(U1-Pad41)
- U1 pad 42: Net-(U1-Pad42) -> unconnected-(U1-Pad42)
- U1 pad 43: Net-(U1-Pad43) -> unconnected-(U1-Pad43)
- U1 pad 44: Net-(U1-Pad44) -> unconnected-(U1-Pad44)
- U1 pad 45: Net-(U1-Pad45) -> unconnected-(U1-Pad45)
- U1 pad 46: Net-(U1-Pad46) -> unconnected-(U1-Pad46)
- U1 pad 47: Net-(U1-Pad47) -> unconnected-(U1-Pad47)
- U1 pad 48: Net-(U1-Pad48) -> unconnected-(U1-Pad48)
- U1 pad 49: Net-(U1-Pad49) -> unconnected-(U1-Pad49)
- U1 pad 5: Net-(U1-Pad5) -> unconnected-(U1-Pad5)
- U1 pad 50: Net-(U1-Pad50) -> /nuCAN1_TX
- U1 pad 51: Net-(U1-Pad51) -> unconnected-(U1-Pad51)
- U1 pad 52: Net-(U1-Pad52) -> /nuCAN1_RX
- U1 pad 53: Net-(U1-Pad53) -> unconnected-(U1-Pad53)
- U1 pad 55: Net-(U1-Pad55) -> /Serial_nu_to_rp
- U1 pad 56: Net-(U1-Pad56) -> unconnected-(U1-Pad56)
- U1 pad 57: Net-(U1-Pad57) -> unconnected-(U1-Pad57)
- U1 pad 58: Net-(U1-Pad58) -> unconnected-(U1-Pad58)
- U1 pad 59: Net-(U1-Pad59) -> unconnected-(U1-Pad59)
- U1 pad 6: Net-(U1-Pad6) -> unconnected-(U1-Pad6)
- U1 pad 60: Net-(U1-Pad60) -> unconnected-(U1-Pad60)
- U1 pad 61: Net-(U1-Pad61) -> unconnected-(U1-Pad61)
- U1 pad 62: Net-(U1-Pad62) -> unconnected-(U1-Pad62)
- U1 pad 63: Net-(U1-Pad63) -> unconnected-(U1-Pad63)
- U1 pad 64: Net-(U1-Pad64) -> unconnected-(U1-Pad64)
- U1 pad 65: Net-(U1-Pad65) -> unconnected-(U1-Pad65)
- U1 pad 66: Net-(U1-Pad66) -> unconnected-(U1-Pad66)
- U1 pad 67: Net-(U1-Pad67) -> unconnected-(U1-Pad67)
- U1 pad 69: Net-(U1-Pad69) -> unconnected-(U1-Pad69)
- U1 pad 7: Net-(U1-Pad7) -> unconnected-(U1-Pad7)
- U1 pad 70: Net-(U1-Pad70) -> unconnected-(U1-Pad70)
- U1 pad 71: Net-(U1-Pad71) -> /Serial_rp_to_nu
- U1 pad 72: Net-(U1-Pad72) -> unconnected-(U1-Pad72)
- U1 pad 73: Net-(U1-Pad73) -> unconnected-(U1-Pad73)
- U1 pad 74: Net-(U1-Pad74) -> unconnected-(U1-Pad74)
- U1 pad 75: Net-(U1-Pad75) -> unconnected-(U1-Pad75)
- U1 pad 76: Net-(U1-Pad76) -> unconnected-(U1-Pad76)
- U1 pad 8: Net-(U1-Pad8) -> unconnected-(U1-Pad8)
- U1 pad 9: Net-(U1-Pad9) -> unconnected-(U1-Pad9)
Routing:
- net /Serial_rp_to_nu: track 0.00 -> 37.6 mm, vias 0 -> 1
- net /Serial_nu_to_rp: track 0.00 -> 15.7 mm
- net +5V: track 0.00 -> 2.54 mm

Commit message: edit some net class
Parts:
- added C1: 22p, Capacitor_SMD:C_0603_1608Metric, F.Cu at (139.7, 119.4)
- added C2: 22p, Capacitor_SMD:C_0603_1608Metric, F.Cu at (162.6, 119.4)
- added H1: MountingHole, MountingHole:MountingHole_3.2mm_M3_Pad_Via, F.Cu at (186.7, 54.6)
- added H2: MountingHole, MountingHole:MountingHole_3.2mm_M3_Pad_Via, F.Cu at (118.1, 54.6)
- added H3: MountingHole, MountingHole:MountingHole_3.2mm_M3_Pad_Via, F.Cu at (101.6, 54.6)
- added H4: MountingHole, MountingHole:MountingHole_3.2mm_M3_Pad_Via, F.Cu at (101.6, 139.7)
- added H5: MountingHole, MountingHole:MountingHole_3.2mm_M3_Pad_Via, F.Cu at (118.1, 139.7)
- added H6: MountingHole, MountingHole:MountingHole_3.2mm_M3_Pad_Via, F.Cu at (186.7, 139.7)
- added J2: Conn_01x04_Female, Connector_JST:JST_XA_S04B-XASK-1_1x04_P2.50mm_Horizontal, F.Cu at (180.3, 102.9)
- added J3: Conn_01x04_Female, Connector_JST:JST_XA_S04B-XASK-1_1x04_P2.50mm_Horizontal, F.Cu at (180.3, 88.9)
- added J4: Conn_01x04_Female, Connector_JST:JST_XA_S04B-XASK-1_1x04_P2.50mm_Horizontal, F.Cu at (180.3, 74.9)
- added R1: 1k, Resistor_SMD:R_0603_1608Metric, F.Cu at (160.0, 105.4)
- added R2: 120, Resistor_SMD:R_0603_1608Metric, F.Cu at (171.4, 109.2)
- added R3: 1k, Resistor_SMD:R_0603_1608Metric, F.Cu at (160.0, 94.0)
- added R4: 120, Resistor_SMD:R_0603_1608Metric, F.Cu at (171.4, 97.8)
- added R5: 1k, Resistor_SMD:R_0603_1608Metric, F.Cu at (158.8, 85.1)
- added R6: 120, Resistor_SMD:R_0603_1608Metric, F.Cu at (171.4, 86.4)
- added U3: MCP2515-xST, Package_SO:TSSOP-20_4.4x6.5mm_P0.65mm, F.Cu at (153.7, 109.2)
- added U4: MCP2551-I-SN, Package_SO:SOIC-8_3.9x4.9mm_P1.27mm, F.Cu at (165.1, 109.2)
- added U5: MCP2551-I-SN, Package_SO:SOIC-8_3.9x4.9mm_P1.27mm, F.Cu at (165.1, 86.4)
- added Y1: Crystal, Crystal:Crystal_SMD_HC49-SD, F.Cu at (151.1, 119.4)
- moved U2 10.9 mm to (165.1, 97.8), turned to 90 degrees
- moved J1 9.92 mm to (141.6, 78.1)
- moved U1 9.92 mm to (118.1, 128.3)
Connections:
- J1 pad 14: unconnected-(J1-Pad14) -> GND
- J1 pad 19: unconnected-(J1-Pad19) -> /rp_MOSI
- J1 pad 20: unconnected-(J1-Pad20) -> GND
- J1 pad 21: unconnected-(J1-Pad21) -> /rp_MISO
- J1 pad 23: unconnected-(J1-Pad23) -> /rp_SCLK
- J1 pad 24: unconnected-(J1-Pad24) -> /rp_~{CS}_MCP2512
- J1 pad 25: unconnected-(J1-Pad25) -> GND
- J1 pad 30: unconnected-(J1-Pad30) -> GND
- J1 pad 34: unconnected-(J1-Pad34) -> GND
- J1 pad 39: unconnected-(J1-Pad39) -> GND
- J1 pad 6: unconnected-(J1-Pad6) -> GND
- J1 pad 9: unconnected-(J1-Pad9) -> GND
- U1 pad 19: unconnected-(U1-Pad19) -> GND
- U1 pad 20: unconnected-(U1-Pad20) -> GND
- U1 pad 22: unconnected-(U1-Pad22) -> GND
- U1 pad 47: unconnected-(U1-Pad47) -> GND
- U1 pad 58: unconnected-(U1-Pad58) -> GND
- U1 pad 6: unconnected-(U1-Pad6) -> +5V
- U1 pad 70: unconnected-(U1-Pad70) -> GND
- U1 pad 8: unconnected-(U1-Pad8) -> GND
- U2 pad 6: unconnected-(U2-Pad6) -> Net-(J3-Pad3)
- U2 pad 7: unconnected-(U2-Pad7) -> Net-(J3-Pad2)
- U2 pad 8: unconnected-(U2-Pad8) -> Net-(R3-Pad1)
Routing:
- net Net-(C1-Pad1): track 0.00 -> 19.3 mm
- net Net-(C2-Pad1): track 0.00 -> 15.0 mm
- net Net-(R1-Pad1): track 0.00 -> 3.39 mm
- net /Serial_nu_to_rp: track 15.7 -> 14.7 mm

Commit message: complete
Parts:
- added C3: 0.1u, Capacitor_SMD:C_0603_1608Metric, F.Cu at (147.3, 105.4)
- added C4: 0.1u, Capacitor_SMD:C_0603_1608Metric, F.Cu at (160.5, 109.2)
- added C5: 0.1u, Capacitor_SMD:C_0603_1608Metric, F.Cu at (165.1, 103.5)
- added C6: 0.1u, Capacitor_SMD:C_0603_1608Metric, F.Cu at (165.1, 91.9)
- added J10: Conn_01x04_Female, Connector_JST:JST_XA_S04B-XASK-1_1x04_P2.50mm_Horizontal, F.Cu at (180.3, 72.4)
- added J11: Conn_01x02_Female, Connector_JST:JST_XA_S02B-XASK-1_1x02_P2.50mm_Horizontal, F.Cu at (180.3, 129.5)
- added J12: Conn_01x02_Female, Connector_JST:JST_XA_S02B-XASK-1_1x02_P2.50mm_Horizontal, F.Cu at (169.7, 133.3)
- added J5: Conn_01x05_Female, Connector_JST:JST_XA_S05B-XASK-1_1x05_P2.50mm_Horizontal, F.Cu at (146.1, 133.3)
- added J6: Conn_01x05_Female, Connector_JST:JST_XA_S05B-XASK-1_1x05_P2.50mm_Horizontal, F.Cu at (156.2, 59.7)
- added J7: Conn_01x05_Female, Connector_JST:JST_XA_S05B-XASK-1_1x05_P2.50mm_Horizontal, F.Cu at (139.7, 59.7)
- added J8: Conn_01x05_Female, Connector_JST:JST_XA_S05B-XASK-1_1x05_P2.50mm_Horizontal, F.Cu at (129.5, 133.3)
- added J9: Conn_02x03_Odd_Even, Connector_PinHeader_2.54mm:PinHeader_2x03_P2.54mm_Vertical, F.Cu at (169.8, 57.7)
- moved J2 15.2 mm to (180.3, 118.1)
- moved J3 15.2 mm to (180.3, 104.1)
- moved J4 15.2 mm to (180.3, 90.2)
- moved H1 0.63 mm to (186.7, 54.0), turned to 180 degrees
- moved H2 0.63 mm to (118.1, 54.0), turned to 180 degrees
- moved H3 0.63 mm to (101.6, 54.0), turned to 180 degrees
- moved H4 0.63 mm to (101.6, 139.1)
- moved H5 0.63 mm to (118.1, 139.1)
- moved H6 0.63 mm to (186.7, 139.1)
Connections:
- J1 pad 1: +3V3 -> unconnected-(J1-Pad1)
- J1 pad 10: /Serial_nu_to_rp -> /UART_RX_rp
- J1 pad 17: +3V3 -> unconnected-(J1-Pad17)
- J1 pad 8: /Serial_rp_to_nu -> /UART_TX_rp
- U1 pad 1: unconnected-(U1-Pad1) -> /nu_PC_10
- U1 pad 2: unconnected-(U1-Pad2) -> /nu_PC_11
- U1 pad 23: unconnected-(U1-Pad23) -> /nu_PC_13
- U1 pad 25: unconnected-(U1-Pad25) -> /nu_PC_14
- U1 pad 27: unconnected-(U1-Pad27) -> /nu_PC_15
- U1 pad 3: unconnected-(U1-Pad3) -> /nu_PC_12
- U1 pad 35: unconnected-(U1-Pad35) -> /nu_PC_2
- U1 pad 36: unconnected-(U1-Pad36) -> /nu_PC_1
- U1 pad 37: unconnected-(U1-Pad37) -> /nu_PC_3
- U1 pad 38: unconnected-(U1-Pad38) -> /nu_PC_0
- U1 pad 39: unconnected-(U1-Pad39) -> /nu_PC_9
- U1 pad 40: unconnected-(U1-Pad40) -> /nu_PC_8
- U1 pad 42: unconnected-(U1-Pad42) -> /nu_PC_6
- U1 pad 44: unconnected-(U1-Pad44) -> /nu_PC_5
- U1 pad 55: /Serial_nu_to_rp -> /UART_TX_nu
- U1 pad 57: unconnected-(U1-Pad57) -> /nu_PC_7
- U1 pad 71: /Serial_rp_to_nu -> /UART_RX_nu
- U1 pad 72: unconnected-(U1-Pad72) -> /nu_PC_4
Routing:
- net +5V: track 2.54 -> 240.8 mm, vias 0 -> 5
- net /nu_PC_10: track 0.00 -> 94.8 mm
- net /nu_PC_11: track 0.00 -> 90.9 mm, vias 0 -> 1
- net /UART_TX_rp: track 0.00 -> 83.2 mm
- net /nuCAN1_TX: track 0.00 -> 81.2 mm, vias 0 -> 1
- net /UART_RX_rp: track 0.00 -> 79.7 mm
- net /nuCAN1_RX: track 0.00 -> 76.6 mm, vias 0 -> 1
- net /nuCAN2_TX: track 0.00 -> 69.4 mm, vias 0 -> 1
- net /UART_TX_nu: track 0.00 -> 50.5 mm
- net /nuCAN2_RX: track 0.00 -> 48.4 mm, vias 0 -> 1
- net /Serial_rp_to_nu: track 37.6 -> 0.00 mm, vias 1 -> 0
- net /nu_PC_5: track 0.00 -> 35.5 mm
- net /rp_~{CS}_MCP2512: track 0.00 -> 34.9 mm, vias 0 -> 1
- net /rp_MOSI: track 0.00 -> 34.8 mm, vias 0 -> 2
- net /nu_PC_6: track 0.00 -> 34.7 mm
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- added copper zone on B.Cu, net GND
- added copper zone on F.Cu, net GND
Other:
- board outline added: 92.7 x 92.7 mm
- board text added: "CAN1_TX PA_12 CAN1_RX PA_11"
- board text added: "CAN2_TX PB_12 CAN2_RX PB_13"
- board text added: "GND PC_11 PC_10 PC_9 PC_8"
- board text added: "GND PC_7 PC_6 PC_5 PC_4"
- board text added: "IO14 TXD"
- board text added: "PA_10 RX"
- board text added: "PC_0 PC_1 PC_2 PC_3 GND"
- board text added: "PC_12 PC_13 PC_14 PC_15 GND"
- board text added: "POWER 5VDC"
- board text added: "RPHAT_nucleo v0 Raspberry Pi CAN HAT with nucleo CAN io designed by paripal https://github.com/paripalpp/RPHAT_nucleo"
- board text added: "nucleo UART1 PB_6 TX"
- board text added: "output"
- board text added: "raspi IO15 RXD"
- board text added: "~{CE0}/GPIO8 MISO0/GPIO9 MOSI0/GPIO10 SCLK0/GPIO11"

Commit message: v1 comp
Parts:
- moved J9 22.2 mm to (183.3, 75.3)
- moved J10 13.9 mm to (174.7, 59.7), turned to 180 degrees
- moved J12 6.35 mm to (163.3, 133.3)
- moved J11 6.15 mm to (175.5, 133.3), turned to 0 degrees
- moved J4 3.05 mm to (180.5, 93.2)
- moved J3 2.92 mm to (180.5, 107.1)
- moved J2 2.80 mm to (180.5, 120.9)
Connections:
- U1 pad 54: /nuCAN2_TX -> /nuCAN2_RX
- U1 pad 68: /nuCAN2_RX -> /nuCAN2_TX
Routing:
- net /UART_TX_rp: track 83.2 -> 111.8 mm
- net /UART_RX_rp: track 79.7 -> 108.3 mm
- net +5V: track 240.8 -> 261.8 mm
- net /nuCAN2_RX: track 48.4 -> 66.2 mm
- net /nuCAN2_TX: track 69.4 -> 51.9 mm, vias 1 -> 2
- net /UART_RX_out: track 14.5 -> 27.5 mm
- net /UART_TX_out: track 14.5 -> 24.6 mm
- net /UART_RX_nu: track 24.7 -> 30.1 mm, vias 0 -> 1
- net /UART_TX_nu: track 50.5 -> 54.2 mm, vias 0 -> 1
- net Net-(J2-Pad2): track 20.2 -> 21.9 mm
- net Net-(J3-Pad2): track 19.4 -> 21.1 mm
- net Net-(J4-Pad2): track 18.0 -> 19.4 mm
- net Net-(J3-Pad3): track 18.0 -> 18.9 mm
- net Net-(J2-Pad3): track 19.0 -> 19.7 mm
- net GND: vias 291 -> 302
Other:
- board text added: "Align headers here"
- board text added: "CAN2_TX PB_13 CAN2_RX PB_12"
- board text added: "IO14 raspi TXD"
- board text added: "IO15 RXD"
- board text added: "J10_2"
- board text added: "J10_3"
- board text added: "Over about 20mm from edge of this board"
- board text added: "PA_10 nucleo RX UART1"
- board text added: "PB_6 TX"
- board text added: "POWER 5VDC x2"
- board text added: "RPHAT_nucleo v1 Raspberry Pi CAN HAT with nucleo CAN io designed by paripal https://github.com/paripalpp/RPHAT_nucleo"
- board text added: "UART output"
- board text added: "for nucleo-144 ST morpho"
- board text added: "for nucleo-144 ST morpho +20"
- board text added: "to use nucleo-144 Align start of headers here"
- board text removed: "CAN2_TX PB_12 CAN2_RX PB_13"
- board text removed: "IO14 TXD"
- board text removed: "PA_10 RX"
- board text removed: "POWER 5VDC"
- board text removed: "RPHAT_nucleo v0 Raspberry Pi CAN HAT with nucleo CAN io designed by paripal https://github.com/paripalpp/RPHAT_nucleo"
- board text removed: "nucleo UART1 PB_6 TX"
- board text removed: "output"
- board text removed: "raspi IO15 RXD"
