File: RPHAT_nucleo.kicad_sch (KiCad schematic)
At the start: 2 parts, among them J1 Raspberry_Pi_2_3, U1 NUCLEO-F446RE

Commit message: on
Parts:
- added U2: MCP2551-I-SN, Package_SO:SOIC-8_3.9x4.9mm_P1.27mm, symbol Interface_CAN_LIN:MCP2551-I-SN
Connections:
- net +3V3: now reaches J1.1 (3V3)
- net +3V3: now also J1.17 (3V3)
- net Serial_nu_to_rp: now reaches J1.10 (GPIO15/RXD)
- net Serial_nu_to_rp: now also U1.55 (PB_6)
- net +5V: now reaches J1.2 (5V)
- net +5V: now also J1.4 (5V), U2.3 (VDD)
- net Serial_rp_to_nu: now reaches J1.8 (GPIO14/TXD)
- net Serial_rp_to_nu: now also U1.71 (PA_10)
- net nuCAN1_TX: now reaches U1.50 (PA_12)
- net nuCAN1_TX: now also U2.1 (TXD)
- net nuCAN1_RX: now reaches U1.52 (PA_11)
- net nuCAN1_RX: now also U2.4 (RXD)
- net nuCAN2_TX: now reaches U1.54 (PB_12)
- net nuCAN2_RX: now reaches U1.68 (PB_13)
- new net GND: U2.2 (VSS)
Changed lines of the file:
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@@
 (kicad_sch (version 20211123) (generator eeschema)
   (paper "A4")
+  (junction (at 106.68 53.34) (diameter 0) (color 0 0 0 0)
+  )
+  (junction (at 99.06 53.34) (diameter 0) (color 0 0 0 0)
+  )
+  (wire (pts (xy 266.7 99.06) (xy 254 99.06))
+    (stroke (width 0) (type default) (color 0 0 0 0))
+  )
+  (wire (pts (xy 96.52 53.34) (xy 99.06 53.34))
+    (stroke (width 0) (type default) (color 0 0 0 0))
+  )
+  (wire (pts (xy 212.09 83.82) (xy 228.6 83.82))
+    (stroke (width 0) (type default) (color 0 0 0 0))
+  )
+  (wire (pts (xy 64.77 68.58) (xy 81.28 68.58))
+    (stroke (width 0) (type default) (color 0 0 0 0))
+  )
+  (wire (pts (xy 96.52 55.88) (xy 96.52 53.34))
+    (stroke (width 0) (type default) (color 0 0 0 0))
+  )
+  (wire (pts (xy 209.55 143.51) (xy 222.25 143.51))
+    (stroke (width 0) (type default) (color 0 0 0 0))
+  )
+  (wire (pts (xy 106.68 53.34) (xy 106.68 55.88))
+    (stroke (width 0) (type default) (color 0 0 0 0))
+  )
+  (wire (pts (xy 104.14 55.88) (xy 104.14 53.34))
+    (stroke (width 0) (type default) (color 0 0 0 0))
+  )
+  (wire (pts (xy 99.06 48.26) (xy 99.06 53.34))
+    (stroke (width 0) (type default) (color 0 0 0 0))
+  )
+  (wire (pts (xy 266.7 81.28) (xy 254 81.28))
+    (stroke (width 0) (type default) (color 0 0 0 0))
+  )
+  (wire (pts (xy 99.06 53.34) (xy 99.06 55.88))
+    (stroke (width 0) (type default) (color 0 0 0 0))
+  )
+  (wire (pts (xy 212.09 104.14) (xy 228.6 104.14))
+    (stroke (width 0) (type default) (color 0 0 0 0))
+  )
+  (wire (pts (xy 234.95 156.21) (xy 234.95 158.75))
+    (stroke (width 0) (type default) (color 0 0 0 0))
+  )
+  (wire (pts (xy 64.77 66.04) (xy 81.28 66.04))
+    (stroke (width 0) (type default) (color 0 0 0 0))
+  )
+  (wire (pts (xy 266.7 78.74) (xy 254 78.74))
+    (stroke (width 0) (type default) (color 0 0 0 0))
+  )
+  (wire (pts (xy 104.14 53.34) (xy 106.68 53.34))
+    (stroke (width 0) (type default) (color 0 0 0 0))
+  )
+  (wire (pts (xy 209.55 140.97) (xy 222.25 140.97))
+    (stroke (width 0) (type default) (color 0 0 0 0))
+  )
+  (wire (pts (xy 106.68 48.26) (xy 106.68 53.34))
+    (stroke (width 0) (type default) (color 0 0 0 0))
+  )
+  (wire (pts (xy 266.7 76.2) (xy 254 76.2))
+    (stroke (width 0) (type default) (color 0 0 0 0))
+  )
+  (wire (pts (xy 234.95 133.35) (xy 234.95 135.89))
+    (stroke (width 0) (type default) (color 0 0 0 0))
+  )
+  (label "Serial_nu_to_rp" (at 64.77 68.58 0)
+    (effects (font (size 1.27 1.27)) (justify left bottom))
+  )
+  (label "nuCAN1_TX" (at 266.7 76.2 180)
+    (effects (font (size 1.27 1.27)) (justify right bottom))
+  )
+  (label "Serial_rp_to_nu" (at 64.77 66.04 0)
+    (effects (font (size 1.27 1.27)) (justify left bottom))
+  )
+  (label "nuCAN1_RX" (at 209.55 143.51 0)
+    (effects (font (size 1.27 1.27)) (justify left bottom))
+  )
+  (label "nuCAN2_RX" (at 266.7 99.06 180)
+    (effects (font (size 1.27 1.27)) (justify right bottom))
+  )
+  (label "Serial_rp_to_nu" (at 212.09 104.14 0)
+    (effects (font (size 1.27 1.27)) (justify left bottom))
+  )
+  (label "Serial_nu_to_rp" (at 212.09 83.82 0)
+    (effects (font (size 1.27 1.27)) (justify left bottom))
+  )
+  (label "nuCAN1_TX" (at 209.55 140.97 0)
+    (effects (font (size 1.27 1.27)) (justify left bottom))
+  )
+  (label "nuCAN1_RX" (at 266.7 78.74 180)
+    (effects (font (size 1.27 1.27)) (justify right bottom))
+  )
+  (label "nuCAN2_TX" (at 266.7 81.28 180)
+    (effects (font (size 1.27 1.27)) (justify right bottom))
+  )
   (symbol (lib_id "Connector:Raspberry_Pi_2_3") (at 101.6 88.9 0) (unit 1)
     (in_bom yes) (on_board yes)
-    (property "Reference" "J1" (id 0) (at 101.6 51.2826 0))
-    (property "Value" "Raspberry_Pi_2_3" (id 1) (at 101.6 53.594 0))
+    (property "Reference" "J1" (id 0) (at 83.82 54.8386 0))
+    (property "Value" "Raspberry_Pi_2_3" (id 1) (at 83.82 57.15 0))
     (property "Footprint" "Boad_dev:RaspberryPi_HAT_Connector_4hole" (id 2) (at 101.6 88.9 0)
       (effects (font (size 1.27 1.27)) hide)
@@
     (pin "76")
   )
+  (symbol (lib_id "power:+5V") (at 234.95 133.35 0) (unit 1)
+    (in_bom yes) (on_board yes) (fields_autoplaced)
+    (property "Reference" "#PWR03" (id 0) (at 234.95 137.16 0)
+      (effects (font (size 1.27 1.27)) hide)
+    )
+    (property "Value" "+5V" (id 1) (at 234.95 129.7455 0))
+    (property "Footprint" "" (id 2) (at 234.95 133.35 0)
+      (effects (font (size 1.27 1.27)) hide)
+    )
+    (property "Datasheet" "" (id 3) (at 234.95 133.35 0)
+      (effects (font (size 1.27 1.27)) hide)
+    )
+    (pin "1")
+  )
+  (symbol (lib_id "power:+5V") (at 99.06 48.26 0) (unit 1)
+    (in_bom yes) (on_board yes) (fields_autoplaced)
+    (property "Reference" "#PWR01" (id 0) (at 99.06 52.07 0)
+      (effects (font (size 1.27 1.27)) hide)
+    )
+    (property "Value" "+5V" (id 1) (at 99.06 44.6555 0))
+    (property "Footprint" "" (id 2) (at 99.06 48.26 0)
+      (effects (font (size 1.27 1.27)) hide)
+    )
+    (property "Datasheet" "" (id 3) (at 99.06 48.26 0)
+      (effects (font (size 1.27 1.27)) hide)
+    )
+    (pin "1")
+  )
+  (symbol (lib_id "Interface_CAN_LIN:MCP2551-I-SN") (at 234.95 146.05 0) (unit 1)
+    (in_bom yes) (on_board yes) (fields_autoplaced)
+    (property "Reference" "U2" (id 0) (at 236.9694 134.4635 0)
+      (effects (font (size 1.27 1.27)) (justify left))
+    )
+    (property "Value" "MCP2551-I-SN" (id 1) (at 236.9694 137.2386 0)
+      (effects (font (size 1.27 1.27)) (justify left))
+    )
+    (property "Footprint" "Package_SO:SOIC-8_3.9x4.9mm_P1.27mm" (id 2) (at 234.95 158.75 0)
+      (effects (font (size 1.27 1.27) italic) hide)
+    )
+    (property "Datasheet" "http://ww1.microchip.com/downloads/en/devicedoc/21667d.pdf" (id 3) (at 234.95 146.05 0)
+      (effects (font (size 1.27 1.27)) hide)
+    )
+    (pin "1")
+    (pin "2")
+    (pin "3")
+    (pin "4")
+    (pin "5")
+    (pin "6")
+    (pin "7")
+    (pin "8")
+  )
+  (symbol (lib_id "power:+3.3V") (at 106.68 48.26 0) (unit 1)
+    (in_bom yes) (on_board yes) (fields_autoplaced)
+    (property "Reference" "#PWR02" (id 0) (at 106.68 52.07 0)
+      (effects (font (size 1.27 1.27)) hide)
+    )
+    (property "Value" "+3.3V" (id 1) (at 106.68 44.6555 0))
+    (property "Footprint" "" (id 2) (at 106.68 48.26 0)
+      (effects (font (size 1.27 1.27)) hide)
+    )
+    (property "Datasheet" "" (id 3) (at 106.68 48.26 0)
+      (effects (font (size 1.27 1.27)) hide)
+    )
+    (pin "1")
+  )
+  (symbol (lib_id "power:GND") (at 234.95 158.75 0) (unit 1)
+    (in_bom yes) (on_board yes) (fields_autoplaced)
+    (property "Reference" "#PWR04" (id 0) (at 234.95 165.1 0)
+      (effects (font (size 1.27 1.27)) hide)
+    )
+    (property "Value" "GND" (id 1) (at 234.95 163.3125 0))
+    (property "Footprint" "" (id 2) (at 234.95 158.75 0)
+      (effects (font (size 1.27 1.27)) hide)
+    )
+    (property "Datasheet" "" (id 3) (at 234.95 158.75 0)
+      (effects (font (size 1.27 1.27)) hide)
+    )
+    (pin "1")
+  )
   (sheet_instances
     (path "/" (page "1"))
   )
   (symbol_instances
+    (path "/50dcc949-9b2f-40bd-8cb1-07d142c192a1"
+      (reference "#PWR01") (unit 1) (value "+5V") (footprint "")
+    )
+    (path "/9f6beb53-a7b4-4e3b-9704-f8c9f23c6ce5"
+      (reference "#PWR02") (unit 1) (value "+3.3V") (footprint "")
+    )
+    (path "/2a54a6e7-bb36-43ca-a6f6-78eff0b07673"
+      (reference "#PWR03") (unit 1) (value "+5V") (footprint "")
+    )
+    (path "/a8e40a2e-59cf-4d65-ba8c-17cb2e89c54e"
+      (reference "#PWR04") (unit 1) (value "GND") (footprint "")
+    )
     (path "/00000000-0000-0000-0000-000061bf1e06"
       (reference "J1") (unit 1) (value "Raspberry_Pi_2_3") (footprint "Boad_dev:RaspberryPi_HAT_Connector_4hole")
@@
       (reference "U1") (unit 2) (value "NUCLEO-F446RE") (footprint "Boad_dev:Nucleo-64_ST_morpho")
     )
-  )
+    (path "/5aa7d921-ee47-49f0-a0db-d8f789a74e8f"
+      (reference "U2") (unit 1) (value "MCP2551-I-SN") (footprint "Package_SO:SOIC-8_3.9x4.9mm_P1.27mm")
+    )
+  )

Commit message: some
Parts:
- added R? (x3): 1k, symbol Device:R
- added U? (x2): MCP2551-I-SN, Package_SO:SOIC-8_3.9x4.9mm_P1.27mm, symbol Interface_CAN_LIN:MCP2551-I-SN
- added U?: MCP2515-xST, Package_SO:TSSOP-20_4.4x6.5mm_P0.65mm, symbol Interface_CAN_LIN:MCP2515-xST
Connections:
- net +5V: now also U?.20 (VDD), U?.3 (VDD), U?.3 (VDD)
- net GND: now also R?.2, R?.2, R?.2, U?.10 (VSS), U?.2 (VSS), U?.2 (VSS)
- net nuCAN2_RX: now also U?.4 (RXD)
- net nuCAN2_TX: now also U?.1 (TXD)
- net rp_MISO: now reaches J1.35 (GPIO19/MISO1)
- net rp_MOSI: now reaches J1.38 (GPIO20/MOSI1)
- net rp_SCLK: now reaches J1.40 (GPIO21/SCLK1)
- net at U2.8 (Rs): now also R?.1
- new net: R?.1, U?.8 (Rs) (x2)
- new net rp_CAN_RX: U?.2 (RXCAN), U?.4 (RXD)
- new net rp_CAN_TX: U?.1 (TXCAN), U?.1 (TXD)
Other:
- moved on the sheet: U2

Commit message: edit some net class
Parts:
- added C1, C2: 22p, Capacitor_SMD:C_0603_1608Metric, symbol Device:C
- added H1, H2, H3, H4, H5, H6: MountingHole, MountingHole:MountingHole_3.2mm_M3_Pad_Via, symbol Mechanical:MountingHole
- added J2, J3, J4: Conn_01x04_Female, Connector_JST:JST_XA_S04B-XASK-1_1x04_P2.50mm_Horizontal, symbol Connector:Conn_01x04_Female
- added R2, R4, R6: 120, Resistor_SMD:R_0603_1608Metric, symbol Device:R
- added Y1: Crystal, Crystal:Crystal_SMD_HC49-SD, symbol Device:Crystal
- R1, R3, R5: renamed from R?; footprint (none) -> Resistor_SMD:R_0603_1608Metric
- gave numbers to parts that had none: 3
Connections:
- net +5V: now also U1.6 (E5V), J2.1 (Pin_1), J3.1 (Pin_1), J4.1 (Pin_1)
- net GND: now also J1.14 (GND), J1.20 (GND), J1.25 (GND), J1.30 (GND), J1.34 (GND), J1.39 (GND), J1.6 (GND), J1.9 (GND), U1.19 (GND), U1.20 (GND), U1.22 (GND), U1.47 (GND), U1.58 (GND), U1.70 (AGND), U1.8 (GND), C1.2, C2.2, J2.4 (Pin_4), J3.4 (Pin_4), J4.4 (Pin_4)
- net rp_MISO: now also J1.21 (MISO0/GPIO9), U3.17 (SO); no longer J1.35 (GPIO19/MISO1)
- net rp_MOSI: now also J1.19 (MOSI0/GPIO10), U3.16 (SI); no longer J1.38 (GPIO20/MOSI1)
- net rp_SCLK: now also J1.23 (SCLK0/GPIO11), U3.14 (SCK); no longer J1.40 (GPIO21/SCLK1)
- net rp_~{CS}_MCP2512: now reaches J1.24 (~{CE0}/GPIO8)
- net rp_~{CS}_MCP2512: now also U3.18 (~{CS})
- net at U4.6 (CANL): now also J2.3 (Pin_3), R2.2
- net at U4.7 (CANH): now also J2.2 (Pin_2), R2.1
- net at U2.6 (CANL): now also J3.3 (Pin_3), R4.2
- net at U2.7 (CANH): now also J3.2 (Pin_2), R4.1
- net at U5.6 (CANL): now also J4.3 (Pin_3), R6.2
- net at U5.7 (CANH): now also J4.2 (Pin_2), R6.1
- net at U3.8 (OSC2): now also C1.1, Y1.1
- net at U3.9 (OSC1): now also C2.1, Y1.2
Other:
- moved on the sheet: R1, R3, U2, U3, U4

Commit message: complete
Parts:
- added C3, C4, C5, C6: 0.1u, Capacitor_SMD:C_0603_1608Metric, symbol Device:C
- added J10: Conn_01x04_Female, Connector_JST:JST_XA_S04B-XASK-1_1x04_P2.50mm_Horizontal, symbol Connector:Conn_01x04_Female
- added J11, J12: Conn_01x02_Female, Connector_JST:JST_XA_S02B-XASK-1_1x02_P2.50mm_Horizontal, symbol Connector:Conn_01x02_Female
- added J5, J6, J7, J8: Conn_01x05_Female, Connector_JST:JST_XA_S05B-XASK-1_1x05_P2.50mm_Horizontal, symbol Connector:Conn_01x05_Female
- added J9: Conn_02x03_Odd_Even, Connector_PinHeader_2.54mm:PinHeader_2x03_P2.54mm_Vertical, symbol Connector_Generic:Conn_02x03_Odd_Even
Connections:
- net +5V: now also C3.1, C4.1, C5.1, C6.1, J10.1 (Pin_1), J11.1 (Pin_1), J12.1 (Pin_1)
- net GND: now also C3.2, C4.2, C5.2, C6.2, J10.4 (Pin_4), J11.2 (Pin_2), J12.2 (Pin_2), J5.5 (Pin_5), J6.5 (Pin_5), J7.5 (Pin_5), J8.5 (Pin_5)
- net nu_PC_10: now reaches U1.1 (PC_10)
- net nu_PC_10: now also J7.3 (Pin_3)
- net nu_PC_11: now reaches U1.2 (PC_11)
- net nu_PC_11: now also J7.4 (Pin_4)
- net nu_PC_13: now reaches U1.23 (PC_13)
- net nu_PC_13: now also J8.2 (Pin_2)
- net nu_PC_14: now reaches U1.25 (PC_14)
- net nu_PC_14: now also J8.3 (Pin_3)
- net nu_PC_15: now reaches U1.27 (PC_15)
- net nu_PC_15: now also J8.4 (Pin_4)
- net nu_PC_12: now reaches U1.3 (PC_12)
- net nu_PC_12: now also J8.1 (Pin_1)
- net nu_PC_2: now reaches U1.35 (PC_2)
- net nu_PC_2: now also J5.3 (Pin_3)
- net nu_PC_1: now reaches U1.36 (PC_1)
- net nu_PC_1: now also J5.2 (Pin_2)
- net nu_PC_3: now reaches U1.37 (PC_3)
- net nu_PC_3: now also J5.4 (Pin_4)
- net nu_PC_0: now reaches U1.38 (PC_0)
- net nu_PC_0: now also J5.1 (Pin_1)
- net nu_PC_9: now reaches U1.39 (PC_9)
- net nu_PC_9: now also J7.2 (Pin_2)
- net nu_PC_8: now reaches U1.40 (PC_8)
- net nu_PC_8: now also J7.1 (Pin_1)
- net nu_PC_6: now reaches U1.42 (PC_6)
- net nu_PC_6: now also J6.3 (Pin_3)
- net nu_PC_5: now reaches U1.44 (PC_5)
- net nu_PC_5: now also J6.2 (Pin_2)
- net nu_PC_7: now reaches U1.57 (PC_7)
- net nu_PC_7: now also J6.4 (Pin_4)
- net nu_PC_4: now reaches U1.72 (PC_4)
- net nu_PC_4: now also J6.1 (Pin_1)
- net +3V3: no longer names the net of J1.1 (3V3)
- net +3V3: no longer J1.17 (3V3)
- net Serial_nu_to_rp renamed UART_RX_rp
- net UART_RX_rp: now also J9.1 (Pin_1); no longer U1.55 (PB_6)
- net Serial_rp_to_nu renamed UART_RX_nu
- net UART_RX_nu: now also J9.4 (Pin_4); no longer J1.8 (GPIO14/TXD)
- new net UART_RX_out: J10.3 (Pin_3), J9.6 (Pin_6)
- new net UART_TX_nu: J9.3 (Pin_3), U1.55 (PB_6)
- new net UART_TX_out: J10.2 (Pin_2), J9.5 (Pin_5)
- new net UART_TX_rp: J1.8 (GPIO14/TXD), J9.2 (Pin_2)

Commit message: v1 comp
Connections:
- net nuCAN2_RX: now also U1.54 (PB_12); no longer U1.68 (PB_13)
- net nuCAN2_TX: now also U1.68 (PB_13); no longer U1.54 (PB_12)
Changed lines of the file:
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@@
     (effects (font (size 1.27 1.27)) (justify left bottom))
   )
-  (label "nuCAN2_RX" (at 266.7 99.06 180)
+  (label "nuCAN2_TX" (at 266.7 99.06 180)
     (effects (font (size 1.27 1.27)) (justify right bottom))
   )
@@
     (effects (font (size 1.27 1.27)) (justify right bottom))
   )
-  (label "nuCAN2_TX" (at 266.7 81.28 180)
+  (label "nuCAN2_RX" (at 266.7 81.28 180)
     (effects (font (size 1.27 1.27)) (justify right bottom))
   )
